Commit message: debugging oarbot

File: dev_ws/src/oarbot-ros/oarbot_description/urdf/base/oarbot_base.gazebo.xacro (robot description, xacro)
@@ -8,6 +8,7 @@
 	      <odometryFrame>odom</odometryFrame>
 	      <odometryRate>50.0</odometryRate>
-	      <robotBaseFrame>base_footprint</robotBaseFrame>
+	      <robotBaseFrame>summit_base_footprint</robotBaseFrame>
 	      <publishTF>true</publishTF>
+	      <legacyModeNS>true</legacyModeNS>
 	    </plugin>
 	  </gazebo>

File: dev_ws/src/oarbot-ros/oarbot_description/urdf/base/oarbot_base.urdf.xacro (robot description, xacro)
@@ -61,4 +61,8 @@
       </geometry>
     </collision>
+    <inertial>
+            <mass value="0.1" />
+            <inertia ixx="0.03" iyy="0.03" izz="0.03" ixy="0.0" ixz="0.0" iyz="0.0" />
+        </inertial>
   </link>
   <joint name="base_to_support" type="fixed">

File: dev_ws/src/oarbot-ros/oarbot_description/urdf/wheels/omni_wheel.urdf.xacro (robot description, xacro)
@@ -6,5 +6,5 @@
   <xacro:property name="wheel_height" value="0.087" />
   <xacro:property name="wheel_mass" value="6.5" /> <!-- in kg-->
-  <xacro:macro name="cylinder_inertia" params="m r h">
+  <xacro:macro name="cylinder_inertial" params="m r h">
     <inertia  ixx="${m*(3*r*r+h*h)/12}" ixy = "0" ixz = "0"
               iyy="${m*r*r/2}" iyz = "0"
@@ -25,11 +25,11 @@
         <xacro:if value="${reflect}">
           <geometry>
-            <mesh filename="package://oarbot_description/meshes/wheels/omni_wheel_1.dae" />
+            <mesh filename="$(find oarbot_description)/meshes/wheels/omni_wheel_1.dae" />
           </geometry>
-          </xacro:if>
-          <xacro:unless value="${reflect}">
-            <geometry>
-              <mesh filename="package://oarbot_description/meshes/wheels/omni_wheel_2.dae" />
-            </geometry>
+        </xacro:if>
+        <xacro:unless value="${reflect}">
+          <geometry>
+            <mesh filename="$(find oarbot_description)/meshes/wheels/omni_wheel_2.dae" />
+          </geometry>
 		    </xacro:unless>
       </visual>
@@ -43,5 +43,7 @@
         <mass value="${wheel_mass}" />
         <origin xyz="0 0 0" />
-        <cylinder_inertia  m="${wheel_mass}" r="${wheel_radius}" h="${wheel_height}" />
+        <inertia  ixx="${wheel_mass}*(3*${wheel_radius}*${wheel_radius}+${wheel_height}*${wheel_height})/12" ixy = "0" ixz = "0"
+              iyy="${wheel_mass}*${wheel_radius}*${wheel_radius}/2" iyz = "0"
+              izz="${wheel_mass}*(3*${wheel_radius}*${wheel_radius}+${wheel_height}*${wheel_height})/12" />
       </inertial>
     </link>
@@ -57,10 +59,10 @@
     </transmission>
     <gazebo reference="${prefix}_wheel_link">
-		<mu1 value="1.0"/>
-		<mu2 value="1.0"/>
-		<kp value="10000000.0" />
-		<kd value="1.0" />
-		<fdir1 value="1 0 0"/>
-        <turnGravityOff>false</turnGravityOff>
+      <mu1 value="1.0"/>
+      <mu2 value="1.0"/>
+      <kp value="10000000.0" />
+      <kd value="1.0" />
+      <fdir1 value="1 0 0"/>
+      <turnGravityOff>false</turnGravityOff>
     </gazebo>
   </xacro:macro>
