Commit message: motion lib video gen

File: dev_ws/src/oarbot-ros/oarbot_description/robot/oarbot.urdf.xacro (robot description, xacro)
@@ -10,4 +10,12 @@
 	<xacro:property name="wheel_offset_z" value="0.0" />
 	<xacro:macro name="robot">
+		<link name="world"/>
+		<joint name="connect_base_and_world" type="prismatic">
+			<child link="summit_base_footprint" />
+			<parent link="world" />
+			<origin xyz="0 0 0" rpy="0 0 0" />
+			<axis xyz="1 0 0"/>
+			<limit effort="1000.0" lower="-100" upper="100" velocity="1000"/>
+		</joint>
 		<xacro:summit_base/>
 		<xacro:omni_wheel prefix="summit_front_right" parent="summit_base_link" reflect="false">

File: dev_ws/src/oarbot-ros/oarbot_description/urdf/base/oarbot_base.urdf.xacro (robot description, xacro)
@@ -9,10 +9,10 @@
 	<!-- BASE FOOTPRINT -->
 		<link name="summit_base_footprint">
-		  <visual>
+		  <!-- <visual>
 			  <origin xyz="0 0 0" rpy="0 0 0" />
 			  <geometry>
 				 <box size="0.001 0.001 0.001" />
 			  </geometry>
-		  </visual>
+		  </visual> -->
 		</link>
 		<joint name="summit_base_footprint_joint" type="fixed">
@@ -51,5 +51,5 @@
     <visual>
       <geometry>
-        <box size="0.15 0.15 0.3"/>
+        <box size="0.15 0.15 0.5"/>
       </geometry>
       <origin rpy="0 0 0" xyz="0 0 -0.15"/>
